Commit message: Update mycobot_pro_450_force_gripper.urdf

File: mycobot_description/urdf/mycobot_pro_450/mycobot_pro_450_force_gripper.urdf (robot description, URDF)
Before this commit: robot firefighter, 16 links, 15 joints
Links:
- link gripper_base: geometry collision box size=0.10 0.05 0.035; visual mesh filename=package://mycobot_description/urdf/mycobot_320_m5_2022/forc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
- link gripper_connection: geometry collision box size=0.05 0.05 0.03; visual mesh filename=package://mycobot_description/urdf/mycobot_320_m5_2022/forc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
- link gripper_left1: geometry collision box size=0.02 0.02 0.055; visual mesh filename=package://mycobot_description/urdf/mycobot_320_m5_2022/forc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
- link gripper_left2: geometry collision box size=0.02 0.055 0.02; visual mesh filename=package://mycobot_description/urdf/mycobot_320_m5_2022/forc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
- link gripper_left3: geometry collision box size=0.02 0.055 0.02; visual mesh filename=package://mycobot_description/urdf/mycobot_320_m5_2022/forc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
- link gripper_right1: geometry collision box size=0.02 0.02 0.055; visual mesh filename=package://mycobot_description/urdf/mycobot_320_m5_2022/forc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
- link gripper_right2: geometry collision box size=0.02 0.055 0.02; visual mesh filename=package://mycobot_description/urdf/mycobot_320_m5_2022/forc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
- link gripper_right3: geometry collision box size=0.02 0.055 0.02; visual mesh filename=package://mycobot_description/urdf/mycobot_320_m5_2022/forc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

Commit message: Update mycobot_pro_450_force_gripper.urdf

File: mycobot_description/urdf/mycobot_pro_450/mycobot_pro_450_force_gripper.urdf (robot description, URDF)
Before this commit: robot firefighter, 16 links, 15 joints
Links:
- link gripper_base: mass 0.05 -> 0.005
- link gripper_connection: mass 1.0 -> 0.1
- link link1: mass 10.0 -> 20.0; geometry collision cylinder length=0.130 radius=0.033; visual mesh filename=package://mycobot_description/urdf/mycobot_pro_450/PRO450_J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
- link link2: mass 5.0 -> 10.0
- link link3: mass 5.0 -> 10.0
- link link4: mass 2.0 -> 5.0
- link link5: mass 2.0 -> 5.0
- link link6: mass 2.0 -> 5.0
