Commit message: Update mycobot_pro_450_force_gripper.urdf

File: mycobotpro450/config/mycobot_pro_450_force_gripper.urdf (robot description, URDF)
Before this commit: robot firefighter, 16 links, 15 joints
Links:
- link link2: mass 10.0 -> 1.0
- link link3: mass 10.0 -> 2.0
- link link4: mass 5.0 -> 1.0
- link link5: mass 5.0 -> 1.0
- link link6: mass 5.0 -> 1.0
Joints:
- joint joint1: limit lower=-2.8797 upper=2.8797 effort=1000.0 velocity=1 -> lower=-2.8274 upper=2.8274 effort=1000.0 velocity=1
- joint joint2: limit lower=-2.0943 upper=2.0943 effort=1000.0 velocity=1 -> lower=-2.1816 upper=2.1816 effort=1000.0 velocity=1
- joint joint3: limit lower=-2.7576 upper=2.7576 effort=1000.0 velocity=1 -> lower=-2.6878 upper=2.6878 effort=1000.0 velocity=1
- joint joint4: limit lower=-2.8797 upper=2.8797 effort=1000.0 velocity=1 -> lower=-2.8274 upper=2.8274 effort=1000.0 velocity=1
- joint joint5: limit lower=-2.8797 upper=2.8797 effort=1000.0 velocity=1 -> lower=-2.8274 upper=2.8274 effort=1000.0 velocity=1
- joint joint6: limit lower=-3.0543 upper=3.0543 effort=1000.0 velocity=1 -> lower=-2.8797 upper=2.8797 effort=1000.0 velocity=1

Commit message: Update mycobot_pro_450_force_gripper.urdf

File: mycobotpro450/config/mycobot_pro_450_force_gripper.urdf (robot description, URDF)
Before this commit: robot firefighter, 16 links, 15 joints
Links:
- link base: geometry collision cylinder length=0.10 radius=0.10; visual mesh filename=package://mycobot_description/urdf/mycobot_pro_450/PRO450_J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
- link link1: geometry collision cylinder length=0.095 radius=0.043; visual mesh filename=package://mycobot_description/urdf/mycobot_pro_450/PRO450_J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
